Commit message: updated length and width of chassis

File: description/gazebo_control.xacro (robot description, xacro)
@@ -6,5 +6,5 @@
             <left_joint>left_wheel_joint</left_joint>
             <right_joint>right_wheel_joint</right_joint>
-            <wheel_separation>0.304</wheel_separation>
+            <wheel_separation>0.32</wheel_separation>
             <wheel_diameter>0.066</wheel_diameter>
             <!-- Limits -->

File: description/robot_core.xacro (robot description, xacro)
@@ -5,6 +5,6 @@
     <!-- <xacro:property name="chassis_height" value="0.12" />
     <xacro:property name="chassis_radius" value="0.12" /> -->
-    <xacro:property name="chassis_length" value="0.304"/>
-    <xacro:property name="chassis_width" value="0.304"/>
+    <xacro:property name="chassis_length" value="0.32"/>
+    <xacro:property name="chassis_width" value="0.32"/>
     <xacro:property name="chassis_height" value="0.076"/>
     <xacro:property name="chassis_mass" value="4.0"/>
